File: HASKEL-Z80/EPROM-27512-GLS27SF512/EPROM-27512-GLS27SF512.kicad_pcb (KiCad board)
At the start: 2 copper layers, 17 x 36.1 mm, 2 parts, among them U101 27512, U102 GLS27SF512

Commit message: update projects
Other:
- board text added: "r2"
- board text removed: "r1"
Changed lines of the file:
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@@
   )
   (page A4)
+  (title_block
+    (date 2023-06-24)
+    (rev r2)
+  )
   (layers
     (0 F.Cu signal)
@@
       (drillshape 0)
       (scaleselection 1)
-      (outputdirectory "r1/"))
+      (outputdirectory "EEPROM-27512-002/"))
   )
   (net 0 "")
@@
       (effects (font (size 1 1) (thickness 0.15)))
     )
+    (fp_line (start 1.255 -1.27) (end 14.985 -1.27) (layer F.Fab) (width 0.1))
+    (fp_line (start 14.985 -1.27) (end 14.985 34.29) (layer F.Fab) (width 0.1))
+    (fp_line (start 14.985 34.29) (end 0.255 34.29) (layer F.Fab) (width 0.1))
+    (fp_line (start 0.255 34.29) (end 0.255 -0.27) (layer F.Fab) (width 0.1))
+    (fp_line (start 0.255 -0.27) (end 1.255 -1.27) (layer F.Fab) (width 0.1))
+    (fp_line (start 6.62 -1.33) (end 1.16 -1.33) (layer F.SilkS) (width 0.12))
+    (fp_line (start 1.16 -1.33) (end 1.16 34.35) (layer F.SilkS) (width 0.12))
+    (fp_line (start 1.16 34.35) (end 14.08 34.35) (layer F.SilkS) (width 0.12))
+    (fp_line (start 14.08 34.35) (end 14.08 -1.33) (layer F.SilkS) (width 0.12))
+    (fp_line (start 14.08 -1.33) (end 8.62 -1.33) (layer F.SilkS) (width 0.12))
+    (fp_line (start -1.05 -1.55) (end -1.05 34.55) (layer F.CrtYd) (width 0.05))
+    (fp_line (start -1.05 34.55) (end 16.3 34.55) (layer F.CrtYd) (width 0.05))
+    (fp_line (start 16.3 34.55) (end 16.3 -1.55) (layer F.CrtYd) (width 0.05))
     (fp_line (start 16.3 -1.55) (end -1.05 -1.55) (layer F.CrtYd) (width 0.05))
-    (fp_line (start 16.3 34.55) (end 16.3 -1.55) (layer F.CrtYd) (width 0.05))
-    (fp_line (start -1.05 34.55) (end 16.3 34.55) (layer F.CrtYd) (width 0.05))
-    (fp_line (start -1.05 -1.55) (end -1.05 34.55) (layer F.CrtYd) (width 0.05))
-    (fp_line (start 14.08 -1.33) (end 8.62 -1.33) (layer F.SilkS) (width 0.12))
-    (fp_line (start 14.08 34.35) (end 14.08 -1.33) (layer F.SilkS) (width 0.12))
-    (fp_line (start 1.16 34.35) (end 14.08 34.35) (layer F.SilkS) (width 0.12))
-    (fp_line (start 1.16 -1.33) (end 1.16 34.35) (layer F.SilkS) (width 0.12))
-    (fp_line (start 6.62 -1.33) (end 1.16 -1.33) (layer F.SilkS) (width 0.12))
-    (fp_line (start 0.255 -0.27) (end 1.255 -1.27) (layer F.Fab) (width 0.1))
-    (fp_line (start 0.255 34.29) (end 0.255 -0.27) (layer F.Fab) (width 0.1))
-    (fp_line (start 14.985 34.29) (end 0.255 34.29) (layer F.Fab) (width 0.1))
-    (fp_line (start 14.985 -1.27) (end 14.985 34.29) (layer F.Fab) (width 0.1))
-    (fp_line (start 1.255 -1.27) (end 14.985 -1.27) (layer F.Fab) (width 0.1))
     (fp_arc (start 7.62 -1.33) (end 6.62 -1.33) (angle -180) (layer F.SilkS) (width 0.12))
     (fp_text user %R (at 7.205399 33.070599) (layer F.Fab)
@@
       (effects (font (size 1 1) (thickness 0.15)))
     )
+    (fp_line (start 4.37 -7.095) (end 5.825 -7.095) (layer F.SilkS) (width 0.12))
+    (fp_line (start 5.825 -7.095) (end 5.825 -5.64) (layer F.SilkS) (width 0.12))
+    (fp_line (start -4.37 7.095) (end -5.825 7.095) (layer F.SilkS) (width 0.12))
+    (fp_line (start -5.825 7.095) (end -5.825 5.64) (layer F.SilkS) (width 0.12))
+    (fp_line (start 4.37 7.095) (end 5.825 7.095) (layer F.SilkS) (width 0.12))
+    (fp_line (start 5.825 7.095) (end 5.825 5.64) (layer F.SilkS) (width 0.12))
+    (fp_line (start -4.37 -7.095) (end -4.652782 -7.095) (layer F.SilkS) (width 0.12))
+    (fp_line (start -4.652782 -7.095) (end -5.825 -5.922782) (layer F.SilkS) (width 0.12))
+    (fp_line (start -5.825 -5.922782) (end -5.825 -5.64) (layer F.SilkS) (width 0.12))
+    (fp_line (start 0 -6.277893) (end 0.5 -6.985) (layer F.Fab) (width 0.1))
+    (fp_line (start 0.5 -6.985) (end 5.715 -6.985) (layer F.Fab) (width 0.1))
+    (fp_line (start 5.715 -6.985) (end 5.715 6.985) (layer F.Fab) (width 0.1))
+    (fp_line (start 5.715 6.985) (end -5.715 6.985) (layer F.Fab) (width 0.1))
+    (fp_line (start -5.715 6.985) (end -5.715 -5.845) (layer F.Fab) (width 0.1))
+    (fp_line (start -5.715 -5.845) (end -4.575 -6.985) (layer F.Fab) (width 0.1))
+    (fp_line (start -4.575 -6.985) (end -0.5 -6.985) (layer F.Fab) (width 0.1))
+    (fp_line (start -0.5 -6.985) (end 0 -6.277893) (layer F.Fab) (width 0.1))
+    (fp_line (start 0 -7.82) (end 4.36 -7.82) (layer F.CrtYd) (width 0.05))
+    (fp_line (start 4.36 -7.82) (end 4.36 -7.23) (layer F.CrtYd) (width 0.05))
+    (fp_line (start 4.36 -7.23) (end 5.96 -7.23) (layer F.CrtYd) (width 0.05))
+    (fp_line (start 5.96 -7.23) (end 5.96 -5.63) (layer F.CrtYd) (width 0.05))
+    (fp_line (start 5.96 -5.63) (end 6.55 -5.63) (layer F.CrtYd) (width 0.05))
+    (fp_line (start 6.55 -5.63) (end 6.55 0) (layer F.CrtYd) (width 0.05))
+    (fp_line (start 0 7.82) (end -4.36 7.82) (layer F.CrtYd) (width 0.05))
+    (fp_line (start -4.36 7.82) (end -4.36 7.23) (layer F.CrtYd) (width 0.05))
+    (fp_line (start -4.36 7.23) (end -5.96 7.23) (layer F.CrtYd) (width 0.05))
+    (fp_line (start -5.96 7.23) (end -5.96 5.63) (layer F.CrtYd) (width 0.05))
+    (fp_line (start -5.96 5.63) (end -6.55 5.63) (layer F.CrtYd) (width 0.05))
+    (fp_line (start -6.55 5.63) (end -6.55 0) (layer F.CrtYd) (width 0.05))
+    (fp_line (start 0 7.82) (end 4.36 7.82) (layer F.CrtYd) (width 0.05))
+    (fp_line (start 4.36 7.82) (end 4.36 7.23) (layer F.CrtYd) (width 0.05))
+    (fp_line (start 4.36 7.23) (end 5.96 7.23) (layer F.CrtYd) (width 0.05))
+    (fp_line (start 5.96 7.23) (end 5.96 5.63) (layer F.CrtYd) (width 0.05))
+    (fp_line (start 5.96 5.63) (end 6.55 5.63) (layer F.CrtYd) (width 0.05))
+    (fp_line (start 6.55 5.63) (end 6.55 0) (layer F.CrtYd) (width 0.05))
+    (fp_line (start 0 -7.82) (end -4.36 -7.82) (layer F.CrtYd) (width 0.05))
+    (fp_line (start -4.36 -7.82) (end -4.36 -7.23) (layer F.CrtYd) (width 0.05))
+    (fp_line (start -4.36 -7.23) (end -4.68 -7.23) (layer F.CrtYd) (width 0.05))
+    (fp_line (start -4.68 -7.23) (end -5.96 -5.95) (layer F.CrtYd) (width 0.05))
+    (fp_line (start -5.96 -5.95) (end -5.96 -5.63) (layer F.CrtYd) (width 0.05))
+    (fp_line (start -5.96 -5.63) (end -6.55 -5.63) (layer F.CrtYd) (width 0.05))
     (fp_line (start -6.55 -5.63) (end -6.55 0) (layer F.CrtYd) (width 0.05))
-    (fp_line (start -5.96 -5.63) (end -6.55 -5.63) (layer F.CrtYd) (width 0.05))
-    (fp_line (start -5.96 -5.95) (end -5.96 -5.63) (layer F.CrtYd) (width 0.05))
-    (fp_line (start -4.68 -7.23) (end -5.96 -5.95) (layer F.CrtYd) (width 0.05))
-    (fp_line (start -4.36 -7.23) (end -4.68 -7.23) (layer F.CrtYd) (width 0.05))
-    (fp_line (start -4.36 -7.82) (end -4.36 -7.23) (layer F.CrtYd) (width 0.05))
-    (fp_line (start 0 -7.82) (end -4.36 -7.82) (layer F.CrtYd) (width 0.05))
-    (fp_line (start 6.55 5.63) (end 6.55 0) (layer F.CrtYd) (width 0.05))
-    (fp_line (start 5.96 5.63) (end 6.55 5.63) (layer F.CrtYd) (width 0.05))
-    (fp_line (start 5.96 7.23) (end 5.96 5.63) (layer F.CrtYd) (width 0.05))
-    (fp_line (start 4.36 7.23) (end 5.96 7.23) (layer F.CrtYd) (width 0.05))
-    (fp_line (start 4.36 7.82) (end 4.36 7.23) (layer F.CrtYd) (width 0.05))
-    (fp_line (start 0 7.82) (end 4.36 7.82) (layer F.CrtYd) (width 0.05))
-    (fp_line (start -6.55 5.63) (end -6.55 0) (layer F.CrtYd) (width 0.05))
-    (fp_line (start -5.96 5.63) (end -6.55 5.63) (layer F.CrtYd) (width 0.05))
-    (fp_line (start -5.96 7.23) (end -5.96 5.63) (layer F.CrtYd) (width 0.05))
-    (fp_line (start -4.36 7.23) (end -5.96 7.23) (layer F.CrtYd) (width 0.05))
-    (fp_line (start -4.36 7.82) (end -4.36 7.23) (layer F.CrtYd) (width 0.05))
-    (fp_line (start 0 7.82) (end -4.36 7.82) (layer F.CrtYd) (width 0.05))
-    (fp_line (start 6.55 -5.63) (end 6.55 0) (layer F.CrtYd) (width 0.05))
-    (fp_line (start 5.96 -5.63) (end 6.55 -5.63) (layer F.CrtYd) (width 0.05))
-    (fp_line (start 5.96 -7.23) (end 5.96 -5.63) (layer F.CrtYd) (width 0.05))
-    (fp_line (start 4.36 -7.23) (end 5.96 -7.23) (layer F.CrtYd) (width 0.05))
-    (fp_line (start 4.36 -7.82) (end 4.36 -7.23) (layer F.CrtYd) (width 0.05))
-    (fp_line (start 0 -7.82) (end 4.36 -7.82) (layer F.CrtYd) (width 0.05))
-    (fp_line (start -0.5 -6.985) (end 0 -6.277893) (layer F.Fab) (width 0.1))
-    (fp_line (start -4.575 -6.985) (end -0.5 -6.985) (layer F.Fab) (width 0.1))
-    (fp_line (start -5.715 -5.845) (end -4.575 -6.985) (layer F.Fab) (width 0.1))
-    (fp_line (start -5.715 6.985) (end -5.715 -5.845) (layer F.Fab) (width 0.1))
-    (fp_line (start 5.715 6.985) (end -5.715 6.985) (layer F.Fab) (width 0.1))
-    (fp_line (start 5.715 -6.985) (end 5.715 6.985) (layer F.Fab) (width 0.1))
-    (fp_line (start 0.5 -6.985) (end 5.715 -6.985) (layer F.Fab) (width 0.1))
-    (fp_line (start 0 -6.277893) (end 0.5 -6.985) (layer F.Fab) (width 0.1))
-    (fp_line (start -5.825 -5.922782) (end -5.825 -5.64) (layer F.SilkS) (width 0.12))
-    (fp_line (start -4.652782 -7.095) (end -5.825 -5.922782) (layer F.SilkS) (width 0.12))
-    (fp_line (start -4.37 -7.095) (end -4.652782 -7.095) (layer F.SilkS) (width 0.12))
-    (fp_line (start 5.825 7.095) (end 5.825 5.64) (layer F.SilkS) (width 0.12))
-    (fp_line (start 4.37 7.095) (end 5.825 7.095) (layer F.SilkS) (width 0.12))
-    (fp_line (start -5.825 7.095) (end -5.825 5.64) (layer F.SilkS) (width 0.12))
-    (fp_line (start -4.37 7.095) (end -5.825 7.095) (layer F.SilkS) (width 0.12))
-    (fp_line (start 5.825 -7.095) (end 5.825 -5.64) (layer F.SilkS) (width 0.12))
-    (fp_line (start 4.37 -7.095) (end 5.825 -7.095) (layer F.SilkS) (width 0.12))
     (fp_text user %R (at -1.9304 -2.6416 90) (layer F.Fab)
       (effects (font (size 1 1) (thickness 0.15)))
@@
     )
   )
-  (gr_text r1 (at 99.0346 74.0156) (layer F.SilkS)
+  (gr_text r2 (at 99.0346 74.0156) (layer F.SilkS)
     (effects (font (size 1 1) (thickness 0.15)))
   )
