File: HASKEL-Z80/PROGRAMMER-GLS27SF512/PROGRAMMER-GLS27SF512.kicad_pcb (KiCad board)
At the start: 2 copper layers, 79 x 110.5 mm, 44 parts, among them J101 Jack-DC, J102 Conn_D24V6F5_5V, K101 MT2-C93402-IC-Relay, K102 MT2-C93402-IC-Relay, Q101 2N7002, Q102 2N7002, Q103 2N7002, Q104 2N7002, SW101 Reset, U101 pico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

Commit message: update projects
Parts:
- R105, R109: value R10K -> R100K
- R107: value R10K -> R1K
Other:
- board text added: "r4"
- board text removed: "r3"

Commit message: EEPROM Programmer r5
Parts:
- R118: value R10K -> R1K
