File: HASKEL-Z80/PROGRAMMER-GLS27SF512/PROGRAMMER-GLS27SF512.sch (KiCad schematic (older format))
At the start: 44 parts, among them J101 Jack-DC, J102 Conn_D24V6F5_5V, K101 MT2-C93402-IC-Relay, K102 MT2-C93402-IC-Relay, Q101 2N7002, Q102 2N7002, Q103 2N7002, Q104 2N7002, SW101 Reset, U101 pico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

Commit message: update projects
Parts:
- R104, R107: value R10K -> R1K
- R105, R109: value R10K -> R100K
Changed lines of the file:
@@
 Sheet 1 1
 Title "GLS27SF512 EEPROM Programmer"
-Date "2023-06-25"
-Rev "3"
+Date "2023-07-02"
+Rev "4"
 Comp ""
 Comment1 ""
@@
 P 3280 7440
 F 0 "R105" V 3185 7500 50  0000 C CNN
-F 1 "R10K" V 3275 7440 50  0000 C CNN
+F 1 "R100K" V 3275 7465 50  0000 C CNN
 F 2 "Resistor_SMD:R_1206_3216Metric_Pad1.30x1.75mm_HandSolder" V 3210 7440 50  0001 C CNN
 F 3 "~" H 3280 7440 50  0001 C CNN
@@
 P 3105 6940
 F 0 "R104" V 3010 7000 50  0000 C CNN
-F 1 "R10K" V 3100 6940 50  0000 C CNN
+F 1 "R1K" V 3100 6940 50  0000 C CNN
 F 2 "Resistor_SMD:R_1206_3216Metric_Pad1.30x1.75mm_HandSolder" V 3035 6940 50  0001 C CNN
 F 3 "~" H 3105 6940 50  0001 C CNN
@@
 P 5350 7415
 F 0 "R109" V 5255 7475 50  0000 C CNN
-F 1 "R10K" V 5345 7415 50  0000 C CNN
+F 1 "R100K" V 5345 7440 50  0000 C CNN
 F 2 "Resistor_SMD:R_1206_3216Metric_Pad1.30x1.75mm_HandSolder" V 5280 7415 50  0001 C CNN
 F 3 "~" H 5350 7415 50  0001 C CNN
@@
 P 5175 6915
 F 0 "R107" V 5080 6975 50  0000 C CNN
-F 1 "R10K" V 5170 6915 50  0000 C CNN
+F 1 "R1K" V 5170 6915 50  0000 C CNN
 F 2 "Resistor_SMD:R_1206_3216Metric_Pad1.30x1.75mm_HandSolder" V 5105 6915 50  0001 C CNN
 F 3 "~" H 5175 6915 50  0001 C CNN
@@
 Wire Wire Line
 	1470 7185 1575 7185
+Connection ~ 1575 7185
+Wire Wire Line
+	1575 7185 1575 7215
 Wire Bus Line
 	1135 5250 7175 5250
@@
 Wire Bus Line
 	8770 1530 8770 4890
-Connection ~ 1575 7185
-Wire Wire Line
-	1575 7185 1575 7215
 $EndSCHEMATC

Commit message: EEPROM Programmer r5
Parts:
- R118: value R10K -> R1K
Changed lines of the file:
@@
 Title "GLS27SF512 EEPROM Programmer"
 Date "2023-07-02"
-Rev "4"
+Rev "5"
 Comp ""
 Comment1 ""
@@
 P 4525 3370
 F 0 "R114" V 4440 3365 50  0000 C CNN
-F 1 "R1K" V 4525 3355 50  0000 C CNN
+F 1 "R1K" V 4520 3370 50  0000 C CNN
 F 2 "Resistor_SMD:R_1206_3216Metric_Pad1.30x1.75mm_HandSolder" V 4455 3370 50  0001 C CNN
 F 3 "~" H 4525 3370 50  0001 C CNN
@@
 P 4850 3155
 F 0 "R118" V 4935 3105 50  0000 L CNN
-F 1 "R10K" V 4850 3050 50  0000 L CNN
+F 1 "R1K" V 4850 3080 50  0000 L CNN
 F 2 "Resistor_SMD:R_1206_3216Metric_Pad1.30x1.75mm_HandSolder" V 4780 3155 50  0001 C CNN
 F 3 "~" H 4850 3155 50  0001 C CNN
